File: Hardware/HackmodWear.sch (EAGLE design)
At the start: 110 parts, among them IC1 MSGEQ7N, Q2 2.5A/30V, U1 ATSAMD21G-A, U2 3.3V, U3 74AHC1G125, U4 DRV2605L, U5 OPA344, U6 ADMP401, U7 APDS-9960, Y1 32.768kHz

Commit message: Adding BOM and gerbers
Parts:
- removed D13, D4: (no value), SparkFun-LED:LED1206
- removed R14, R27: 330, SparkFun-Resistors:330OHM-0603-1/10W-1%
- added J41, J42, J43, J44, J45, J46, J47, J48, J49, J50, J51, J52, J53, J54, J55, J56, J57, J58, J59, J60, J61, J62, J63, J64, J65, J66, J67, J68, J69, J70, J71, J72, J73, J74, J75, J76: (no value), SparkFun-Connectors:CONN_01
- added S2: (no value), SparkFun-Switches:SWITCH-SPDT-SMD-RIGHT-ANGLE
Connections:
- removed net DI1: J26.1, J32.1
- removed net INT: J40.1, R10.1, U7.INT
- removed net VL: C12.+, C13.1, J24.1, R29.1, U7.LEDA
- net 3.3V: now also J17.1, J44.1, J45.1, J47.1, J52.1, J56.1, J57.1, J60.1, J62.1, J64.1, J66.1, J68.1, J70.1, J73.1, J76.1; no longer D13.A, D4.A
- net A0: no longer IC1.DCOUT, J37.1, J5.1
- net A1: no longer J10.1
- net A2: no longer J11.1
- net A3: now also IC1.DCOUT, J10.1, J37.1; no longer J3.1
- net D0/RXI: no longer J21.1
- net D1/TXO: no longer J19.1
- net D10/SS: no longer J17.1
- net D11/MOSI: no longer J14.1
- net D12/MISO: no longer J16.1
- net D13/SCK: no longer J15.1
- net D2: now also D2.DI, J14.1, J42.1, J53.1
- net D5: now also C12.+, C13.1, J24.1, J3.1, R29.1, U7.LEDA
- net D6: now also J26.1, J32.1
- net D7: now also J40.1, J5.1, R10.1, U7.INT
- net DO: now also J41.1, J54.1; no longer D2.DI
- net DOUT: now also J48.1, J50.1
- net GND: now also J11.1, J19.1, J43.1, J46.1, J49.1, J51.1, J55.1, J58.1, J59.1, J61.1, J63.1, J65.1, J67.1, J69.1, J72.1, J75.1; no longer R14.1, R27.1
- net N$21: now also J71.1, S2.S; no longer D4.C, R27.2
- net N$8: now also J21.1, J74.1; no longer D13.C, R14.2
- net SCL: now also J15.1
- net SDA: now also J16.1
- net VIN: now also S2.P
Other:
- note added: "FUN LEDs"
- note added: "LEDs"
- note removed: "PA12 is SPI MISO (on SPI header)."
- note removed: "PA13 is DGI GPIO0 (goes to EDBG)."
- note removed: "PA5 is A4"
- note removed: "PB10/11 are MOSI/SCK to SPI header."
- note removed: "PB2 is A5"
- note removed: "PB22/23 are TXD/RXD to the EDBG"
- note removed: "SAMD21"
- moved on the sheet: C1, C10, C11, C12, C13, C14, C15, C16, C17, C18, C19, C2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
