File: Hardware/HackmodWear_workingcopy.brd (EAGLE design)
At the start: 99.9 x 104.8 mm, 181 parts, among them Q1 ZXMP6A13F, Q2 NTR4101P, U1 ATSAMD21G-A, U2 3.3V, U5 OPA344, U6 ADMP401, U7 APDS-9960, Y1 32.768kHz

Commit message: pusging before Eagle decides to crash again losing hours of work - thanks eagle 9 for nothing
Parts:
- moved U$53 7.39 mm to (85.6, 76.5)
- moved J57 7.35 mm to (84.1, 70.5)
- moved J50 7.31 mm to (87.7, 76.8)
- moved U$58 7.11 mm to (81.9, 69.7)
- moved J76 0.50 mm to (60.6, 69.6)
- moved S2 0.49 mm to (62.2, 93.5)
- moved J75 0.49 mm to (62.2, 72.5), turned to 240 degrees
- moved J56 0.48 mm to (34.5, 81.0)
- moved J25 0.45 mm to (32.3, 95.5)
- moved J45 0.44 mm to (13.1, 77.1)
- moved J49 0.42 mm to (86.1, 91.9)
- moved J34 0.41 mm to (28.7, 76.9)
- moved J6 0.40 mm to (36.1, 78.1)
- moved J43 0.40 mm to (30.4, 92.3)
- moved J73 0.38 mm to (44.6, 67.4)
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Routing:
- net DOUT: track 35.6 -> 29.0 mm, vias 1 -> 0
- net GND: track 36.6 -> 41.9 mm, vias 117 -> 118
- net 3.3V: track 448.6 -> 444.0 mm, vias 10 -> 11
- net N$21: track 4.84 -> 5.57 mm
- net DO: track 26.4 -> 25.7 mm
- net D7: track 96.2 -> 95.5 mm
- net D9: track 62.0 -> 61.5 mm
- net VIN: track 7.51 -> 8.03 mm
Other:
- outline, holes or cut-outs redrawn

Commit message: Adding gerbers
Parts:
- added U$15, U$17, U$18, U$24, U$25, U$27, U$28, U$34, U$59: (no value), buzzard_labels(4):#15
- added U$29: (no value), buzzard_labels(4):AUD0
- added U$30: (no value), buzzard_labels(3):RST15
- added U$60: (no value), buzzard_labels(2):SDA4
- added U$61, U$62, U$63, U$64, U$65, U$66, U$67, U$68, U$69: (no value), buzzard_labels(4):#16
- added U$70: (no value), buzzard_labels(2):GND2
- added U$71, U$72: (no value), buzzard_labels(2):SCL5
- added U$73: (no value), buzzard_labels(4):INT14
- added U$74, U$75, U$76: (no value), buzzard_labels(4):PT2
- added U$77: (no value), buzzard_labels(4):D211
- added U$78: (no value), buzzard_labels(4):LED4
- added U$79: (no value), buzzard_labels(4):SAMD2112
- added U$80: (no value), buzzard_labels(4):VIBE1
- added U$81: (no value), buzzard_labels(5):NC0
- moved U$2 26.9 mm to (55.8, 68.9)
- moved U$16 2.68 mm to (44.3, 40.3)
- moved U$12 0.42 mm to (36.4, 78.5)
- moved U$19 0.31 mm to (48.8, 40.4)
- moved U$50 0.28 mm to (85.8, 89.6)
- moved U$55 0.26 mm to (70.9, 71.3)
- moved U$48 0.25 mm to (87.6, 86.5)
- moved U$4 0.24 mm to (34.7, 85.1)
- moved U$33 0.24 mm to (34.5, 81.3)
- moved U$7 0.24 mm to (41.3, 69.9)
- moved U$51 0.23 mm to (70.9, 95.0)
- moved U$49 0.23 mm to (73.0, 91.4)
- moved U$21 0.23 mm to (45.6, 59.8)
- moved U$53 0.22 mm to (85.7, 76.4)
- moved U$13 0.19 mm to (52.6, 68.8)
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Connections:
- new net 1: J24.P$1
- new net LEDA: C13.1, R29.1, U7.5
- net D5: no longer C13.1, J24.P$1, R29.1, U7.5
Routing:
- net D5: track 195.2 -> 6.94 mm, vias 2 -> 0
- net LEDA: track 0.00 -> 12.7 mm, vias 0 -> 3
Other:
- board text removed: "+"
- board text removed: "-"
- board text removed: "To Do: 10/7 Fix sew taps on top part NEW BOM!! Silk Order Parts gerbers Order Boards DRC - ugh"
