File: Hardware/HackmodWear_workingcopy.sch (EAGLE design)
At the start: 133 parts, among them Q1 ZXMP6A13F, Q2 NTR4101P, U1 ATSAMD21G-A, U2 3.3V, U5 OPA344, U6 ADMP401, U7 APDS-9960, Y1 32.768kHz

Commit message: Adding gerbers
Connections:
- new net 1: J24.1
- new net LEDA: C13.1, R29.1, U7.LEDA
- net D5: no longer C13.1, J24.1, R29.1, U7.LEDA
Changed lines of the file:
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@@
 <label x="-137.16" y="-114.3" size="1.27" layer="95" xref="yes"/>
-</segment>
-<segment>
-<pinref part="J24" gate="G$1" pin="1"/>
-<wire x1="-190.5" y1="-335.28" x2="-187.96" y2="-335.28" width="0.1524" layer="91"/>
-<label x="-187.96" y="-335.28" size="1.27" layer="95" xref="yes"/>
-</segment>
-<segment>
-<pinref part="U7" gate="G$1" pin="LEDA"/>
-<wire x1="-144.78" y1="-368.3" x2="-157.48" y2="-368.3" width="0.1524" layer="91"/>
-<pinref part="C13" gate="G$1" pin="1"/>
-<wire x1="-157.48" y1="-368.3" x2="-175.26" y2="-368.3" width="0.1524" layer="91"/>
-<wire x1="-175.26" y1="-368.3" x2="-175.26" y2="-370.84" width="0.1524" layer="91"/>
-<wire x1="-175.26" y1="-368.3" x2="-180.34" y2="-368.3" width="0.1524" layer="91"/>
-<label x="-180.34" y="-368.3" size="1.27" layer="95" rot="R180" xref="yes"/>
-<junction x="-175.26" y="-368.3"/>
-<pinref part="R29" gate="G$1" pin="1"/>
-<junction x="-157.48" y="-368.3"/>
 </segment>
 </net>
@@
 </segment>
 </net>
+<net name="LEDA" class="0">
+<segment>
+<pinref part="U7" gate="G$1" pin="LEDA"/>
+<wire x1="-144.78" y1="-368.3" x2="-157.48" y2="-368.3" width="0.1524" layer="91"/>
+<pinref part="R29" gate="G$1" pin="1"/>
+<pinref part="C13" gate="G$1" pin="1"/>
+<wire x1="-175.26" y1="-368.3" x2="-175.26" y2="-370.84" width="0.1524" layer="91"/>
+<wire x1="-157.48" y1="-368.3" x2="-175.26" y2="-368.3" width="0.1524" layer="91"/>
+<junction x="-157.48" y="-368.3"/>
+</segment>
+</net>
+<net name="1" class="0">
+<segment>
+<pinref part="J24" gate="G$1" pin="1"/>
+<wire x1="-190.5" y1="-335.28" x2="-187.96" y2="-335.28" width="0.1524" layer="91"/>
+<label x="-187.96" y="-335.28" size="1.27" layer="95" xref="yes"/>
+</segment>
+</net>
