File: Hardware/HackmodWear_workingcopy3.brd (EAGLE design)
At the start: 99.9 x 104.8 mm, 126 parts, among them Q1 ZXMP6A13F, U1 ATSAMD21G-A, U2 3.3V, U5 OPA344, U6 ADMP401, U7 APDS-9960, Y1 32.768kHz

Commit message: continuing trace routing
Routing:
- net 3.3V: track 291.2 -> 301.9 mm
Changed lines of the file:
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@@
 <wire x1="61.4925" y1="83.5025" x2="59.96305" y2="80.3148" width="0" layer="19" extent="1-1"/>
 <wire x1="43.21625" y1="79.78375" x2="48.21625" y2="83.78375" width="0" layer="19" extent="1-1"/>
+<via x="68.73875" y="59.21375" extent="1-16" drill="0.381"/>
+<via x="77.62875" y="59.53125" extent="1-16" drill="0.381"/>
+<via x="75.2475" y="56.03875" extent="1-16" drill="0.381"/>
+<via x="71.4375" y="56.515" extent="1-16" drill="0.381"/>
+<via x="33.3375" y="60.0075" extent="1-16" drill="0.381"/>
+<via x="23.8125" y="59.69" extent="1-16" drill="0.381"/>
+<via x="26.9875" y="56.35625" extent="1-16" drill="0.381"/>
 </signal>
 <signal name="3.3V">
@@
 <wire x1="33" y1="57" x2="32.5325" y2="57.4675" width="0.254" layer="1"/>
 <wire x1="32.5325" y1="57.4675" x2="31.75" y2="57.4675" width="0.254" layer="1"/>
-<wire x1="73.1925" y1="57.69625" x2="74.20625" y2="57.69625" width="0.254" layer="1"/>
-<wire x1="74.20625" y1="57.69625" x2="74.77125" y2="58.26125" width="0.254" layer="1"/>
 <wire x1="24.57125" y1="57.01625" x2="25.34" y2="57.785" width="0.254" layer="1"/>
 <wire x1="25.34" y1="57.785" x2="26.9875" y2="57.785" width="0.254" layer="1"/>
@@
 <wire x1="27" y1="60" x2="26.9875" y2="59.9875" width="0.254" layer="1"/>
 <wire x1="26.9875" y1="59.9875" x2="26.9875" y2="57.785" width="0.254" layer="1"/>
+<wire x1="71.4375" y1="60.3849" x2="71.4375" y2="59.055" width="0.254" layer="1"/>
+<wire x1="71.4375" y1="59.055" x2="70.64375" y2="58.26125" width="0.254" layer="1"/>
+<wire x1="70.64375" y1="58.26125" x2="69.69125" y2="57.30875" width="0.254" layer="1"/>
+<wire x1="69.69125" y1="57.30875" x2="69.69125" y2="57.30875" width="0.254" layer="1"/>
+<wire x1="68.7783" y1="56.93925" x2="69.32175" y2="56.93925" width="0.254" layer="1"/>
+<wire x1="69.32175" y1="56.93925" x2="69.69125" y2="57.30875" width="0.254" layer="1"/>
+<wire x1="73.1925" y1="57.69625" x2="71.20875" y2="57.69625" width="0.254" layer="1"/>
+<wire x1="71.20875" y1="57.69625" x2="70.64375" y2="58.26125" width="0.254" layer="1"/>
+<wire x1="73.1925" y1="57.69625" x2="76.6049" y2="57.69625" width="0.254" layer="1"/>
+<wire x1="76.6049" y1="57.69625" x2="77.156596875" y2="57.144553125" width="0.254" layer="1"/>
+<wire x1="77.156596875" y1="57.144553125" x2="77.156596875" y2="56.977203125" width="0.254" layer="1"/>
+<wire x1="77.156596875" y1="56.977203125" x2="77.3852" y2="56.7486" width="0.254" layer="1"/>
+<wire x1="77.3852" y1="56.7486" x2="77.55255" y2="56.7486" width="0.254" layer="1"/>
 <wire x1="88.10625" y1="88.8111" x2="85.456946875" y2="81.41228125" width="0" layer="19" extent="1-1"/>
-<wire x1="84.90585" y1="70.3453" x2="83.7175" y2="79.21625" width="0" layer="19" extent="1-1"/>
-<wire x1="71.4375" y1="60.3849" x2="77.5" y2="67" width="0" layer="19" extent="1-1"/>
-<wire x1="74.77125" y1="58.26125" x2="71.4375" y2="60.3849" width="0" layer="19" extent="1-1"/>
-<wire x1="77.55255" y1="56.7486" x2="74.20625" y2="57.69625" width="0" layer="19" extent="1-1"/>
-<wire x1="68.7783" y1="56.93925" x2="73.1925" y2="57.69625" width="0" layer="19" extent="1-1"/>
+<wire x1="81.21" y1="70.79" x2="83.7175" y2="79.21625" width="0" layer="19" extent="1-1"/>
+<wire x1="71.4375" y1="60.3849" x2="71.509503125" y2="67" width="0" layer="19" extent="1-1"/>
 <wire x1="60.59939375" y1="69.570215625" x2="69.1769" y2="69.332603125" width="0" layer="19" extent="1-1"/>
 <wire x1="28.65755" y1="76.89215" x2="34.4551" y2="80.9625" width="0" layer="19" extent="16-16"/>

Commit message: UPdated route out
Routing:
- net 3.3V: track 301.9 -> 375.3 mm, vias 9 -> 10
- net DO: track 0.00 -> 25.0 mm
- net N$16: track 0.00 -> 18.2 mm, vias 0 -> 2
- net N$14: track 0.00 -> 7.37 mm
- net D9: track 22.8 -> 21.2 mm
Other:
- outline, holes or cut-outs redrawn

Commit message: Final Board layout
Parts:
- moved C1 0.67 mm to (51.7, 73.2)
Routing:
- net 3.3V: track 375.3 -> 492.3 mm, vias 10 -> 11
- net GND: track 0.00 -> 46.0 mm, vias 13 -> 70
- net D2: track 65.5 -> 108.9 mm, vias 1 -> 3
- net D9: track 21.2 -> 59.2 mm
- net D7: track 34.4 -> 52.9 mm
- net A3: track 67.8 -> 83.3 mm
- net SCL: track 66.0 -> 75.4 mm
- net SDA: track 62.1 -> 70.7 mm
- net VDDCORE: track 12.3 -> 18.1 mm
- net N$15: track 0.00 -> 3.35 mm
- net !RESET: track 19.8 -> 19.2 mm
Other:
- outline, holes or cut-outs redrawn

Commit message: updated per awesome peer review
Parts:
- added C16, C27, C28, C29: 1.0uF, SparkFun-Capacitors:0603
- added R3, R5: 4.7k, SparkFun-Resistors:0603
- moved R10 7.52 mm to (54.1, 56.0)
- moved R29 7.51 mm to (61.5, 50.0)
- moved U5 1.71 mm to (51.6, 41.3)
- moved U6 1.71 mm to (51.4, 34.9)
- moved C14 1.71 mm to (48.6, 39.1)
- moved C17 1.71 mm to (56.3, 42.1)
- moved C18 1.71 mm to (55.2, 36.7)
- moved C19 1.71 mm to (60.5, 42.1)
- moved C20 1.71 mm to (44.0, 42.6)
- moved R11 1.71 mm to (44.0, 40.8)
- moved R12 1.71 mm to (58.4, 42.1)
- moved R13 1.71 mm to (44.0, 37.1)
- moved R9 1.71 mm to (44.0, 38.9)
Connections:
- net 3.3V: now also R3.2, R5.1
- net GND: now also C16.2, C27.2, C28.2, C29.2
- net LEDA: now also C16.1, C27.1, C28.1, C29.1
- net SCL: now also R5.2
- net SDA: now also R3.1
Routing:
- net LEDA: track 5.96 -> 19.1 mm
- net 3.3V: track 492.3 -> 504.9 mm, vias 11 -> 10
- net SCL: track 75.4 -> 79.1 mm
- net SDA: track 70.7 -> 73.9 mm, vias 2 -> 3
- net D7: track 52.9 -> 50.4 mm
- net A3: track 83.3 -> 85.0 mm
- net D6: track 12.6 -> 11.1 mm
- net GND: vias 70 -> 73
Other:
- outline, holes or cut-outs redrawn

Commit message: final board/sch
Parts:
- added U$1: (no value), BottomSilk_noLabels_300dpi#png:BOTTOMSILK_NOLABELS_300DPI#PNG
- added U$2: (no value), TopSilk_300dpi#01#png:TOPSILK_300DPI#01#PNG
Changed lines of the file:
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@@
 <grid distance="0.01" unitdist="mm" unit="mm" style="lines" multiple="1" display="yes" altdistance="0.01" altunitdist="mm" altunit="mm"/>
 <layers>
-<layer number="1" name="Top" color="4" fill="1" visible="yes" active="yes"/>
+<layer number="1" name="Top" color="4" fill="1" visible="no" active="yes"/>
 <layer number="2" name="Route2" color="1" fill="3" visible="no" active="yes"/>
 <layer number="15" name="Route15" color="4" fill="6" visible="no" active="yes"/>
-<layer number="16" name="Bottom" color="1" fill="1" visible="yes" active="yes"/>
-<layer number="17" name="Pads" color="2" fill="1" visible="yes" active="yes"/>
-<layer number="18" name="Vias" color="2" fill="1" visible="yes" active="yes"/>
-<layer number="19" name="Unrouted" color="6" fill="1" visible="yes" active="yes"/>
+<layer number="16" name="Bottom" color="1" fill="1" visible="no" active="yes"/>
+<layer number="17" name="Pads" color="2" fill="1" visible="no" active="yes"/>
+<layer number="18" name="Vias" color="2" fill="1" visible="no" active="yes"/>
+<layer number="19" name="Unrouted" color="6" fill="1" visible="no" active="yes"/>
 <layer number="20" name="Dimension" color="15" fill="1" visible="no" active="yes"/>
-<layer number="21" name="tPlace" color="7" fill="1" visible="no" active="yes"/>
-<layer number="22" name="bPlace" color="14" fill="1" visible="no" active="yes"/>
-<layer number="23" name="tOrigins" color="15" fill="1" visible="yes" active="yes"/>
-<layer number="24" name="bOrigins" color="15" fill="1" visible="no" active="yes"/>
+<layer number="21" name="tPlace" color="7" fill="1" visible="yes" active="yes"/>
+<layer number="22" name="bPlace" color="14" fill="1" visible="yes" active="yes"/>
+<layer number="23" name="tOrigins" color="15" fill="1" visible="no" active="yes"/>
+<layer number="24" name="bOrigins" color="15" fill="1" visible="yes" active="yes"/>
 <layer number="25" name="tNames" color="7" fill="1" visible="no" active="yes"/>
 <layer number="26" name="bNames" color="7" fill="1" visible="no" active="yes"/>
@@
 <attribute name="VALUE" x="54.782" y="50.15" size="0.6096" layer="27" font="vector" ratio="20" rot="R90" align="top-center"/>
 </element>
+<element name="U$1" library="BottomSilk_noLabels_300dpi#png" package="BOTTOMSILK_NOLABELS_300DPI#PNG" value="" x="49.95" y="52.32" rot="MR0"/>
+<element name="U$2" library="TopSilk_300dpi#01#png" package="TOPSILK_300DPI#01#PNG" value="" x="50.68" y="52.39"/>
 </elements>
 <signals>

Commit message: Cleaning stuff
Other:
- board text added: "https://creativecommons.org/licenses/by-nc-sa/4.0/legalcode This license lets others remix, tweak, and build upon your work non-commercially, and although their new works must also acknowledge you and be non-commercial, they don’t have to license their derivative works on the same terms."
