File: Hardware/HackmodWear_workingcopy3.sch (EAGLE design)
At the start: 126 parts, among them Q1 ZXMP6A13F, U1 ATSAMD21G-A, U2 3.3V, U5 OPA344, U6 ADMP401, U7 APDS-9960, Y1 32.768kHz

Commit message: updated per awesome peer review
Parts:
- added C16, C27, C28, C29: 1.0uF, SparkFun-Capacitors:1.0UF-0603-16V-10%
- added R3, R5: 4.7k, SparkFun-Resistors:4.7KOHM-0603-1/10W-1%
Connections:
- net 3.3V: now also R3.2, R5.1
- net GND: now also C16.2, C27.2, C28.2, C29.2
- net LEDA: now also C16.1, C27.1, C28.1, C29.1
- net SCL: now also R5.2
- net SDA: now also R3.1

Commit message: Cleaning stuff
Other:
- note added: "https://creativecommons.org/licenses/by-nc-sa/4.0/legalcode This license lets others remix, tweak, and build upon your work non-commercially, and although their new works must also acknowledge you and be non-commercial, they don’t have to license their derivative works on the same terms."
Changed lines of the file:
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@@
 <?xml version="1.0" encoding="utf-8"?>
 <!DOCTYPE eagle SYSTEM "eagle.dtd">
-<eagle version="9.2.0">
+<eagle version="9.1.0">
 <drawing>
 <settings>
@@
 <text x="-396.24" y="7.62" size="12.7" layer="97">FUN LEDs</text>
 <circle x="198.12" y="-88.9" radius="101.6" width="3.81" layer="97"/>
+<text x="-15.24" y="-251.46" size="5.08" layer="97">https://creativecommons.org/licenses/by-nc-sa/4.0/legalcode
+This license lets others remix, tweak, and build upon your work
+non-commercially, and although their new works must also
+acknowledge you and be non-commercial, they don’t have to
+ license their derivative works on the same terms.</text>
 </plain>
 <instances>
