File: Bat/SmallBatSAO.brd (EAGLE design)
At the start: 65.3 x 34.5 mm, 0 parts

Commit message: Bat Badge
Parts:
- added BT1: LIPO-OUTLINE100, SparkFun-Batteries:LIPO-110
- added C1, C2, C3, C5: 0.1uF, SparkFun-Capacitors:0603
- added J1: (no value), SparkFun-Connectors:JST-2-SMD
- added LED5, LED6, LED7: (no value), PLCC4_reverse-mount_led:PLCC4_SMD_REVERSE_MOUNT_LED
- added Q1, Q2, Q3: 310mA/60V/1.6Ω, SparkFun-DiscreteSemi:SOT323
- added R1, R2, R3: 330, SparkFun-Resistors:0603
- added R4: 10k, SparkFun-Resistors:0603
- added S1: MOMENTARY-SWITCH-SPST-SMD-4.6X2.8MM, SparkFun-Switches:TACTILE_SWITCH_SMD_4.6X2.8MM
- added U$17: ATTINY85_SOIC, ATTiny85:SOIC-8
Connections:
- new net B: LED5.P$3, LED6.P$3, LED7.P$4, Q1.3
- new net BLUE: Q1.1, R1.1
- new net BUTTON: R4.1, S1.3, S1.4, U$17.2
- new net G: LED5.P$2, LED6.P$2, LED7.P$2, Q2.3
- new net GND: C1.2, C2.2, C3.2, C5.2, J1.2, Q1.2, Q2.2, Q3.2, S1.1, S1.2, U$17.4
- new net MISO/GREEN: Q2.1, R2.2
- new net MOSI/RED: Q3.1, R3.2
- new net N$1: R2.1, U$17.6
- new net N$10: R1.2, U$17.3
- new net N$3: R3.1, U$17.5
- new net R: LED5.P$4, LED6.P$4, LED7.P$3, Q3.3
- new net RESET: U$17.1
- new net SCK: U$17.7
- new net VDD: C1.1, C2.1, C3.1, C5.1, J1.1, LED5.P$1, LED6.P$1, LED7.P$1, R4.2, U$17.8
Routing:
- net VDD: track 0.00 -> 114.1 mm, vias 0 -> 2
- net R: track 0.00 -> 61.2 mm, vias 0 -> 2
- net B: track 0.00 -> 57.2 mm, vias 0 -> 5
- net G: track 0.00 -> 53.8 mm, vias 0 -> 4
- net BUTTON: track 0.00 -> 41.0 mm, vias 0 -> 1
- net BLUE: track 0.00 -> 27.7 mm, vias 0 -> 2
- net MISO/GREEN: track 0.00 -> 16.9 mm, vias 0 -> 2
- net MOSI/RED: track 0.00 -> 12.0 mm, vias 0 -> 2
- net N$3: track 0.00 -> 10.4 mm
- net N$1: track 0.00 -> 10.1 mm
- net N$10: track 0.00 -> 6.75 mm
- added copper zone on layer 1, net GND
- added copper zone on layer 16, net GND

Commit message: Eagle 9 giving me trouble again
Parts:
- removed BT1: LIPO-OUTLINE100, SparkFun-Batteries:LIPO-110
- removed J1: (no value), SparkFun-Connectors:JST-2-SMD
- removed LED7: (no value), PLCC4_reverse-mount_led:PLCC4_SMD_REVERSE_MOUNT_LED
- removed Q1, Q2, Q3: 310mA/60V/1.6Ω, SparkFun-DiscreteSemi:SOT323
- added J2: (no value), SparkFun-Connectors:JST-2-SMD
- added LED1: (no value), PLCC4_reverse-mount_led:PLCC4_SMD_REVERSE_MOUNT_LED
- added S2: (no value), SparkFun-Switches:SWITCH_DPDT_SMD_AYZ0202
- moved C5 17.7 mm to (31.6, 20.7)
- moved R4 13.6 mm to (34.0, 20.7)
- moved C2 11.5 mm to (36.4, 20.7)
- moved C1 3.27 mm to (44.4, 27.9), turned to 270 degrees
- moved S1 0.32 mm to (34.6, 16.5)
Connections:
- removed net BLUE: Q1.1, R1.1
- removed net MISO/GREEN: Q2.1, R2.2
- removed net MOSI/RED: Q3.1, R3.2
- new net VBATT: J2.2, S2.3
- net B: now also LED1.P$3, R2.2; no longer LED7.P$4, Q1.3
- net G: now also LED1.P$2, R3.2; no longer LED7.P$2, Q2.3
- net GND: now also J2.1; no longer J1.2, Q1.2, Q2.2, Q3.2
- net R: now also LED1.P$4, R1.1; no longer LED7.P$3, Q3.3
- net VDD: now also LED1.P$1, S2.2; no longer J1.1, LED7.P$1
Routing:
- net VDD: track 114.1 -> 0.00 mm, vias 2 -> 0
- net BLUE: track 27.7 -> 0.00 mm, vias 2 -> 0
- net BUTTON: track 41.0 -> 14.1 mm, vias 1 -> 0
- net R: track 61.2 -> 44.2 mm, vias 2 -> 0
- net MISO/GREEN: track 16.9 -> 0.00 mm, vias 2 -> 0
- net MOSI/RED: track 12.0 -> 0.00 mm, vias 2 -> 0
- net B: track 57.2 -> 46.7 mm, vias 5 -> 0
- net N$3: track 10.4 -> 0.00 mm
- net N$1: track 10.1 -> 0.00 mm
- net G: track 53.8 -> 46.0 mm, vias 4 -> 0
- net N$10: track 6.75 -> 0.00 mm
- net GND: track 0.00 -> 5.05 mm, vias 13 -> 0
- removed copper zone on layer 16, net GND
Other:
- outline, holes or cut-outs redrawn
- board text added: "+"
- board text added: "_"
- board text added: "blue"
- board text added: "btn"
- board text added: "gnd"
- board text added: "miso/g"
- board text added: "mosi/r"
- board text added: "rst"
- board text added: "sck"
- board text added: "vcc"

Commit message: batt changes
Parts:
- added C4: 0.1uF, SparkFun-Capacitors:0603
- moved C2 17.6 mm to (33.5, 3.35), turned to 0 degrees
- moved C5 7.77 mm to (38.2, 16.6)
- moved R4 5.00 mm to (31.0, 16.7)
- moved S2 1.68 mm to (34.4, 7.91), turned to 180 degrees
- moved C3 0.19 mm to (14.2, 30.5), turned to 180 degrees
Connections:
- net GND: now also C4.2
- net VBATT: now also C4.1
Routing:
- net VDD: track 0.00 -> 115.1 mm, vias 0 -> 4
- net VBATT: track 0.00 -> 43.3 mm, vias 0 -> 2
- net G: track 46.0 -> 72.2 mm, vias 0 -> 2
- net B: track 46.7 -> 61.8 mm, vias 0 -> 3
- net R: track 44.2 -> 58.9 mm, vias 0 -> 3
- net BUTTON: track 14.1 -> 28.7 mm, vias 0 -> 1
- net N$3: track 0.00 -> 10.6 mm
- net N$1: track 0.00 -> 10.0 mm
- net N$10: track 0.00 -> 5.54 mm
- net GND: track 5.05 -> 0.00 mm, vias 0 -> 16
- added copper zone on layer 16, net GND
