File: Bat/SmallBatSAO.sch (EAGLE design)
At the start: 18 parts, among them Q1 310mA/60V/1.6Ω, Q2 310mA/60V/1.6Ω, Q3 310mA/60V/1.6Ω

Commit message: Eagle 9 giving me trouble again
Parts:
- removed BT1: LIPO-OUTLINE100, SparkFun-Batteries:LIPO-OUTLINE100
- removed J1: (no value), SparkFun-Connectors:CONN_02-JST-2MM-SMT
- removed LED7: (no value), PLCC4_reverse-mount_led:PLCC4_REVERSE_MOUNT
- removed Q1, Q2, Q3: 310mA/60V/1.6Ω, SparkFun-DiscreteSemi:MOSFET-NCH-2N7002PW
- added J2: (no value), SparkFun-Connectors:JST_2MM_MALE
- added LED1: (no value), PLCC4_reverse-mount_led:PLCC4_REVERSE_MOUNT
- added S2: (no value), SparkFun-Switches:SWITCH-SPDT-SMD-AYZ0202
Connections:
- removed net BLUE: Q1.G, R1.1
- removed net MISO/GREEN: Q2.G, R2.2
- removed net MOSI/RED: Q3.G, R3.2
- new net VBATT: J2.+, S2.S
- net B: now also LED1.P$3, R2.2; no longer LED7.P$1, Q1.D
- net G: now also LED1.P$2, R3.2; no longer LED7.P$2, Q2.D
- net GND: now also J2.-; no longer J1.1, Q1.S, Q2.S, Q3.S
- net R: now also LED1.P$1, R1.1; no longer LED7.P$3, Q3.D
- net VDD: now also LED1.P$4, S2.P; no longer J1.2, LED7.P$4

Commit message: batt changes
Parts:
- added C4: 0.1uF, SparkFun-Capacitors:0.1UF-0603-25V-(+80/-20%)
Connections:
- net GND: now also C4.2
- net VBATT: now also C4.1
Changed lines of the file:
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@@
 <part name="S2" library="SparkFun-Switches" deviceset="SWITCH-SPDT" device="-SMD-AYZ0202"/>
 <part name="SUPPLY2" library="SparkFun-PowerSymbols" deviceset="VDD" device=""/>
+<part name="C4" library="SparkFun-Capacitors" deviceset="0.1UF" device="-0603-25V-(+80/-20%)" value="0.1uF"/>
 </parts>
 <sheets>
@@
 <instance part="S2" gate="1" x="45.72" y="33.02" rot="MR0"/>
 <instance part="SUPPLY2" gate="VDD" x="50.8" y="36.576"/>
+<instance part="C4" gate="G$1" x="87.63" y="25.908"/>
 </instances>
 <busses>
@@
 <pinref part="C2" gate="G$1" pin="2"/>
 <wire x1="68.58" y1="23.368" x2="68.58" y2="20.32" width="0.1524" layer="91"/>
-<wire x1="68.58" y1="20.32" x2="68.58" y2="15.24" width="0.1524" layer="91"/>
+<wire x1="68.58" y1="20.32" x2="68.58" y2="17.78" width="0.1524" layer="91"/>
 <junction x="68.58" y="20.32"/>
 <pinref part="GND8" gate="1" pin="GND"/>
+<pinref part="C4" gate="G$1" pin="2"/>
+<wire x1="68.58" y1="17.78" x2="68.58" y2="15.24" width="0.1524" layer="91"/>
+<wire x1="87.63" y1="23.368" x2="87.63" y2="17.78" width="0.1524" layer="91"/>
+<wire x1="87.63" y1="17.78" x2="68.58" y2="17.78" width="0.1524" layer="91"/>
+<junction x="68.58" y="17.78"/>
 </segment>
 </net>
@@
 <wire x1="38.1" y1="30.48" x2="40.64" y2="30.48" width="0.1524" layer="91"/>
 </segment>
-</net>
+<segment>
+<pinref part="C4" gate="G$1" pin="1"/>
+<wire x1="87.63" y1="30.988" x2="87.63" y2="38.1" width="0.1524" layer="91"/>
+<wire x1="87.63" y1="38.1" x2="88.9" y2="38.1" width="0.1524" layer="91"/>
+<label x="88.9" y="38.1" size="1.27" layer="95" xref="yes"/>
+</segment>
+</net>
